Commit message: add hinge

File: urdf/diff_drive.urdf (robot description, URDF)
Before this commit: robot diff_drive_robot, 8 links, 7 joints
Links:
- added link left_hinge_link, mass 0.5; collision cylinder length=0.5 radius=0.03; visual cylinder length=0.5 radius=0.03
- added link right_hinge_link, mass 0.5; collision cylinder length=0.5 radius=0.03; visual cylinder length=0.5 radius=0.03
Joints:
- added joint left_hinge: type revolute, parent base_link, child left_hinge_link, origin xyz=0 0.2 0.1 rpy=0 0 0, axis 1 0 0, limit lower=-2.217 upper=0 effort=20 velocity=1
- added joint right_hinge: type revolute, parent base_link, child right_hinge_link, origin xyz=0 -0.2 0.1 rpy=0 0 0, axis 1 0 0, limit lower=0 upper=2.217 effort=20 velocity=1
